File: uRinks/uRinks_v4.0.sch (EAGLE design)
At the start: 136 parts, among them IC1 LM1117-3.3, IC2 STM32F405RGT6, IC3 LM4040B10, IC4 4051PW, IC5 MCP6002, IC6 WM8731, IC7 MCP6004-I_ST, IC8 TL072, J1 WQP-PJ301M-12_JACK, J10 WQP-PJ301M-12_JACK, J2 WQP-PJ301M-12_JACK, J3 WQP-PJ301M-12_JACK, J4 WQP-PJ301M-12_JACK, J5 WQP-PJ301M-12_JACK, J6 WQP-PJ301M-12_JACK, J7 WQP-PJ301M-12_JACK, J8 WQP-PJ301M-12_JACK, J9 WQP-PJ301M-12_JACK, Q1 8MHz, Q2 MMBT3904, Q3 12.288MHz

Commit message: last version uRinks
Parts:
- added H1: MOUNT-HOLE3.2, holes:MOUNT-HOLE3.2
- C10, C11, C13, C14, C15, C17, C18, C19, C20, C25, C26, C27, C30, C31, C35, C37, C39, C42, C43, C44, C45, C47, C48, C49, C6, C7, C9: device rcl:C-USC0603 -> atom_v1_1_board_2:PARTS_AMAN_CAPACITOR
- C28, C29, C36: device resistor:C-USC0603 -> atom_v1_1_board_2:PARTS_AMAN_CAPACITOR
- R1, R11, R12, R13, R14, R15, R16, R17, R18, R19, R20, R27, R3, R33, R38, R39, R4, R40, R41, R42, R43, R44, R5, R51, R53, R54, R57, R60, R61, R8: device rcl:R-US_R0603 -> atom_v1_1_board_2:PARTS_AMAN_RESISTOR
- R21, R22, R23, R24, R25, R26, R31, R32, R34, R35, R36, R37, R50: device resistor:R-US_R0603 -> atom_v1_1_board_2:PARTS_AMAN_RESISTOR
- R55, R56: value 1.0k -> 1k; device rcl:R-US_R0603 -> atom_v1_1_board_2:PARTS_AMAN_RESISTOR
Connections:
- net AREF_-10: now also R12.1, R15.1, R20.1; no longer R12.2, R15.2, R20.2
- net BRIGHTNESS_CV: now also R18.2; no longer R18.1
- net GND: now also R27.1; no longer R27.2
- net IN_1: now also R27.2; no longer R27.1
- net N$1: now also R19.1; no longer R19.2
- net N$14: now also R13.1, R14.2, R15.2; no longer R13.2, R14.1, R15.1
- net N$18: now also R54.2; no longer R54.1
- net N$2: now also R18.1, R19.2, R20.2; no longer R18.2, R19.1, R20.1
- net N$21: now also R54.1; no longer R54.2
- net N$23: now also R43.1; no longer R43.2
- net N$25: now also R42.1, R43.2, R44.2; no longer R42.2, R43.1, R44.1
- net N$28: now also R42.2, R56.1; no longer R42.1, R56.2
- net N$29: now also R56.2; no longer R56.1
- net N$3: now also R14.1; no longer R14.2
- net N$31: now also R40.1; no longer R40.2
- net N$32: now also R39.2, R40.2, R41.1; no longer R39.1, R40.1, R41.2
- net N$33: now also R41.2, R55.1; no longer R41.1, R55.2
- net N$34: now also R55.2; no longer R55.1
- net N$45: now also R39.1; no longer R39.2
- net N$46: now also R44.1; no longer R44.2
- net VEE: now also R12.2; no longer R12.1
- net V_OCT_CV: now also R13.2; no longer R13.1
Other:
- note added: "Olivier Gillet"
- note added: "ol.gillet@gmail.com"
- note removed: "Codex-Modulex"
- note removed: "Original design by: Olivier Gillet of Mutable Instruments"
- note removed: "info@codex-modulex.com"
- moved on the sheet: D3, R12, R13, R14, R15, R18, R19, R20, R27, R39, R40, R41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
